File: capstone_core/core_system.kicad_sch (KiCad schematic)
At the start: 10 parts, among them U2 LSM6DSVTR, U3 ZED F9P GNSS & RTK Module, U4 PCA9306USG

Commit message: putting all footprints in Capstone Footprints Library
Parts:
- U3: footprint ZED-F9P:Zed F9P -> Capstone Footprints:ZED-F9P
- U4: footprint US8_2P40X2P10_ONS -> Capstone Footprints:LevelShift_US8_2P40X2P10_ONS
Changed lines of the file:
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@@
 			)
 		)
-		(property "Footprint" "US8_2P40X2P10_ONS"
+		(property "Footprint" "Capstone Footprints:LevelShift_US8_2P40X2P10_ONS"
 			(at 148.59 133.35 0)
 			(effects
@@
 			)
 		)
-		(property "Footprint" "ZED-F9P:Zed F9P"
+		(property "Footprint" "Capstone Footprints:ZED-F9P"
 			(at 222.25 58.42 0)
 			(effects
