File: capstone_core/capstone_core.kicad_sch (KiCad schematic)
At the start: 22 parts, among them J1 Conn_02x20_Odd_Even, J2 2x5 CONN DSUB-PCB, J3 2x5 CONN DSUB-PCB, J4 Conn_01x02_Socket, J5 Conn_01x02_Socket, J6 Conn_01x02_Socket, U1 ZED F9P GNSS & RTK Module

Commit message: Core PCB. Revision 1.0
Parts:
- removed J5: Conn_01x02_Socket, Capstone Footprints:1x2_CONN_SD-43650-010_02_MOL, symbol Connector:Conn_01x02_Socket
- added C1, C2: 22uF/35V, Capacitor_SMD:C_0805_2012Metric_Pad1.18x1.45mm_HandSolder, symbol Device:C
- added C10: 100uF/16V, Capstone Footprints:CAP_100uF_16V_16SEPC100M_TSS, symbol Device:C_Polarized
- added C11: 0.1uF/10V, Capacitor_SMD:C_0603_1608Metric_Pad1.08x0.95mm_HandSolder, symbol Device:C
- added C12, C25: 680uF/35V, Capstone Footprints:CAP_680uF_35V_UHW1V681MPD6, symbol Device:C_Polarized
- added C13, C15, C17, C18, C19, C20: 22uF/10V, Capacitor_SMD:C_0805_2012Metric_Pad1.18x1.45mm_HandSolder, symbol Device:C
- added C14, C26, C27, C33, C7, C8, C9: 1uF/35V, Capacitor_SMD:C_0603_1608Metric_Pad1.08x0.95mm_HandSolder, symbol Device:C
- added C16, C28, C29, C4: 10nF/50V, Capacitor_SMD:C_0603_1608Metric_Pad1.08x0.95mm_HandSolder, symbol Device:C
- added C21: 2.2uF/6.3V, Capacitor_SMD:C_0603_1608Metric_Pad1.08x0.95mm_HandSolder, symbol Device:C
- added C22: 15pF/50V, Capacitor_SMD:C_0603_1608Metric_Pad1.08x0.95mm_HandSolder, symbol Device:C
- added C23, C30: 330uF/35V, Capstone Footprints:CAP_330uF_35V_UCL1V331MNL1GS-L, symbol Device:C_Polarized
- added C24: 220uF/10V, Capstone Footprints:CAP_100uF_16V_16SEPC100M_TSS, symbol Device:C_Polarized
- added C3: 1uF/35V, Capacitor_SMD:C_0805_2012Metric_Pad1.18x1.45mm_HandSolder, symbol Device:C
- added C31, C32: 4.7uF/6.3V, Capacitor_SMD:C_0603_1608Metric_Pad1.08x0.95mm_HandSolder, symbol Device:C
- added C5, C6: 10uF/25V, Capacitor_SMD:C_0805_2012Metric_Pad1.18x1.45mm_HandSolder, symbol Device:C
- added D1, D2, D3: 50V/3A, Diode_SMD:D_SMC_Handsoldering, symbol Device:D_Schottky
- added H4: MountingHole, MountingHole:MountingHole_2.7mm, symbol Mechanical:MountingHole
- added L1, L3, L4: 33uH, Capstone Footprints:IND_33uH_3A_CDRH127NP-330MC, symbol Device:L
- added L2: 6.8uH, Capstone Footprints:IND_6.8uH_CB_DRA127, symbol Device:L
- added R1, R2: 47k, Resistor_SMD:R_0603_1608Metric_Pad0.98x0.95mm_HandSolder, symbol Device:R_US
- added R3: 100k, Resistor_SMD:R_0603_1608Metric_Pad0.98x0.95mm_HandSolder, symbol Device:R_US
- added R4: 23.2k, Resistor_SMD:R_0603_1608Metric_Pad0.98x0.95mm_HandSolder, symbol Device:R_US
- added R5: 4.9k, Resistor_SMD:R_0603_1608Metric_Pad0.98x0.95mm_HandSolder, symbol Device:R_US
- added RV1: 2k, Capstone Footprints:POT_2k_PV36W202C01B00, symbol Device:R_Potentiometer_Trim_US
- added TP12, TP13, TP14, TP15: TestPoint, Capstone Footprints:testpoint_1.0mm_hole, symbol Connector:TestPoint
- added U3: LM2676SX-12/NOPB, Capstone Footprints:LM2676SX-12-L, symbol Capstone Symbols:LM2676SX-12_NOPB
- added U4: LM62460QRPHRQ1, Capstone Footprints:LM62460QRPHRQ1, symbol Capstone Symbols:LM62460QRPHRQ1
- added U5, U7: LM2596S-5.0, Capstone Footprints:LM2596S-5, symbol Capstone Symbols:LM2596S-5.0
- added U6: LP2985-18DBVR, Capstone Footprints:LP2985-18DBVR, symbol Capstone Symbols:LP2985-18DBVR
- added U8, U9: LP2985-33DBVR, Capstone Footprints:LP2985-33DBVR, symbol Capstone Symbols:LP2985-33DBVR
- H1: footprint MountingHole:MountingHole_2.5mm -> MountingHole:MountingHole_2.7mm
- H2: renamed from H3; footprint MountingHole:MountingHole_2.5mm -> MountingHole:MountingHole_2.7mm
- H3: renamed from H2; footprint MountingHole:MountingHole_2.5mm -> MountingHole:MountingHole_2.7mm
- J1: footprint Capstone Footprints:2x20_CONN_3020-40-0100-00_CNC -> Capstone Footprints:RPI_Hat_B+
- TP1, TP10, TP11, TP2, TP3, TP5, TP6, TP7, TP8, TP9: footprint TestPoint:TestPoint_THTPad_D1.0mm_Drill0.5mm -> Capstone Footprints:testpoint_1.0mm_hole
- TP4: value TestPoint -> +LBW_3V3; footprint TestPoint:TestPoint_THTPad_D1.0mm_Drill0.5mm -> Capstone Footprints:testpoint_1.0mm_hole
- U2: renamed from U1; symbol ZED_F9P:ZED-F9P -> Capstone Symbols:ZED-F9P
- renumbered J6 to J5, U2 to U1
Connections:
- net +12V: now also C10.1, L1.2, R1.1, U3.6 (FB)
- net +1V8: now also C21.1, U6.5 (VOUT)
- net +3V3: now also C14.1, C31.1, U6.1 (VIN), U6.3 (ON/~OFF), U8.5 (VOUT)
- net +CORE_5V: now also C23.1, C26.1, L3.2, U5.4 (FEEDBACK), U8.1 (VIN), U8.3 (ON/~{OFF})
- net +LBW_3V3: now also C32.1, TP13.1, U9.5 (VOUT)
- net +LBW_5V: now also C27.1, C30.1, L4.2, TP12.1, U7.4 (FEEDBACK), U9.1 (VIN), U9.3 (ON/~{OFF})
- net +PI_5V: now also J1.2 (Pin_2), J1.4 (Pin_4), C13.1, C15.1, C17.1, C18.1, C19.1, C20.1, C24.1, C33.1, L2.2, R2.2, R3.1, R5.1, U4.5 (BIAS)
- net +V_BATT: now also C1.1, C12.1, C2.1, C25.1, C3.1, C5.1, C6.1, C8.1, C9.1, U3.2 (IN), U4.13 (EN), U4.14 (VIN), U4.2 (VIN), U5.1 (VIN), U7.1 (VIN)
- net GND: now also C1.2, C10.2, C12.2, C13.2, C14.2, C15.2, C16.2, C17.2, C18.2, C19.2, C2.2, C20.2, C21.2, C23.2, C24.2, C25.2, C26.2, C27.2, C28.2, C29.2, C3.2, C30.2, C31.2, C32.2, C33.2, C5.2, C6.2, C7.2, C8.2, C9.2, D1.2 (A), D2.2 (A), D3.2 (A), RV1.2, RV1.3, TP14.1, TP15.1, U3.4 (GND), U3.8 (TAB), U4.1 (PGND), U4.12 (SYNC_MODE), U4.15 (PGND), U4.8 (AGND), U5.3 (GROUND), U5.5 (~{ON}/OFF), U5.6 (GND_TAB), U6.2 (GND), U7.3 (GROUND), U7.5 (~{ON}/OFF), U7.6 (GND_TAB), U8.2 (GND), U9.2 (GND)
- new net: C4.2, U3.3 (CB)
- new net: R1.2, U3.7 (ON/~OFF)
- new net: C28.1, U8.4 (BYPASS)
- new net: C29.1, U9.4 (BYPASS)
- new net: C22.2, R3.2, R4.1, U4.7 (FB)
- new net: R4.2, RV1.1
- new net: C16.1, U6.4 (BYPASS)
- new net: C11.1, L2.1, U4.16 (SW)
- new net: C11.2, U4.3 (RBOOT), U4.4 (CBOOT)
- new net: C7.1, U4.11 (SpSp), U4.6 (VCC), U4.9 (RT)
- new net: C22.1, R5.2
- new net: R2.1, U4.10 (RESET)
- new net 12V_SW: C4.1, D1.1 (K), L1.1, U3.1 (SW)
- new net CORE_5V_SW: D2.1 (K), L3.1, U5.2 (OUTPUT)
- new net LBW_5V_SW: D3.1 (K), L4.1, U7.2 (OUTPUT)
- no-connect marks 35 -> 34
Other:
- note added: "1.8V Linear Regulator"
- note added: "3.3V Linear Regulator"
- note added: "Buck regulate to 12V/3A for HBW"
- note added: "Buck regulate to 5V/3A for LBW"
- note added: "Buck regulate to 5V/3A for core"
- note added: "ZED-F9P GNSS Receiver"
- note removed: "Pi Power, 5V/5A"
- moved on the sheet: J1, J2, J4, J5, TP10, TP11, TP4, TP5, TP9, U1, U2

Commit message: Added 3D models, changed C12 and C25 to shorter capacitor. Fixed library paths to be relative to KiCad project directory
Parts:
- C12, C25: footprint Capstone Footprints:CAP_680uF_35V_UHW1V681MPD6 -> Capstone Footprints:CAP_680uF_35V_EEHZS1V681UV
- J1: footprint Capstone Footprints:RPI_Hat_B+ -> Capstone Footprints:PI_Connector
Changed lines of the file:
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@@
 			)
 		)
-		(property "Footprint" "Capstone Footprints:RPI_Hat_B+"
+		(property "Footprint" "Capstone Footprints:PI_Connector"
 			(at 49.53 48.26 0)
 			(effects
@@
 			)
 		)
-		(property "Footprint" "Capstone Footprints:CAP_680uF_35V_UHW1V681MPD6"
+		(property "Footprint" "Capstone Footprints:CAP_680uF_35V_EEHZS1V681UV"
 			(at 304.4952 92.71 0)
 			(effects
@@
 			)
 		)
-		(property "Footprint" "Capstone Footprints:CAP_680uF_35V_UHW1V681MPD6"
+		(property "Footprint" "Capstone Footprints:CAP_680uF_35V_EEHZS1V681UV"
 			(at 191.4652 92.71 0)
 			(effects
